Commit message: Pushing

File: kinova_description/urdf/kinect_stand.urdf.xacro (robot description, xacro)
@@ -18,5 +18,5 @@
                          cam_pz="0.0"
                          cam_or="0.0"
-                         cam_op="${40*PI/180}"
+                         cam_op="${45*PI/180}"
                          cam_oy="0.0"/>
 </robot>

File: kinova_description/urdf/objects/table.xacro (robot description, xacro)
@@ -98,5 +98,5 @@
 	<link name="tabletop_corner"/>
 	<joint name="set_tabletop_relto_corner" type="fixed">
-		<origin xyz="0.42 0.3 0" rpy="0 0 -0.76" /> <!-- exact 45 degrees of -0.785398163397458 does not match the real table -->
+		<origin xyz="0.42 0.0055 0" rpy="0 0 -1.56" /> <!-- exact 45 degrees of -0.785398163397458 does not match the real table -->
 		<parent link="tabletop_ontop"/>
 		<child link="tabletop_corner"/>

File: kinova_description/urdf/stand/properties.xacro (robot description, xacro)
@@ -6,5 +6,5 @@
     <xacro:property name="footMass" value="5.0"/>
     <xacro:property name="standRadius" value="0.03"/>
-    <xacro:property name="standHeight" value="1.3"/>
+    <xacro:property name="standHeight" value="1.1"/>
     <xacro:property name="standMass" value="0.5"/>
 </robot>
