Commit message: Prev

File: kinova_description/urdf/kinect/kinect.xacro (robot description, xacro)
@@ -4,18 +4,18 @@
         <!-- Kinect sensor URDF part, cf. https://github.com/turtlebot/turtlebot
         and there turtlebot_description/urdf/sensors/kinect.xacro -->
-        <joint name="${name}_depth_joint" type="fixed">
+        <joint name="${name}_rgb_joint" type="fixed">
             <parent link="${parent}"/>
-            <child link="${name}_depth_frame"/>
-            <origin xyz="0 -0.025 0" rpy="0 0 0"/>
+            <child link="${name}_rgb_frame"/>
+            <origin xyz="${cam_px} ${cam_py} ${cam_pz}" rpy="${cam_or} ${cam_op} ${cam_oy}"/>
         </joint>
-        <link name="${name}_depth_frame"/>
-        <joint name="${name}_depth_optical_joint" type="fixed">
-            <parent link="${name}_depth_frame"/>
-            <child link="${name}_depth_optical_frame"/>
+        <link name="${name}_rgb_frame"/>
+        <joint name="${name}_rgb_optical_joint" type="fixed">
+            <parent link="${name}_rgb_frame"/>
+            <child link="${name}_rgb_optical_frame"/>
             <origin xyz="0 0 0" rpy="-1.57 0 -1.57"/>
         </joint>
-        <link name="${name}_depth_optical_frame"/>
+        <link name="${name}_rgb_optical_frame"/>
         <joint name="${name}_joint" type="fixed">
-            <parent link="${name}_depth_frame"/>
+            <parent link="${name}_rgb_frame"/>
             <child link="${name}_link"/>
             <origin xyz="0 -0.0125 -0.016" rpy="0 0 0"/>
@@ -42,4 +42,16 @@
             </inertial>
         </link>
+        <joint name="${name}_depth_joint" type="fixed">
+            <parent link="${name}_rgb_frame"/>
+            <child link="${name}_depth_frame"/>
+            <origin xyz="0 -0.025 0" rpy="0 0 0"/>
+        </joint>
+        <link name="${name}_depth_frame"/>
+        <joint name="${name}_depth_optical_joint" type="fixed">
+            <parent link="${name}_depth_frame"/>
+            <child link="${name}_depth_optical_frame"/>
+            <origin xyz="0 0 0" rpy="-1.57 0 -1.57"/>
+        </joint>
+        <link name="${name}_depth_optical_frame"/>
         <!-- Not sure why in a macro arguments cannot be passed to an
         associated .gazebo.xacro file... -->
@@ -51,13 +63,13 @@
                 <update_rate>30.0</update_rate>
                 <camera>
-                    <horizontal_fov>${50*M_PI/180.0}</horizontal_fov>
+                    <horizontal_fov>${70.0*3.14/180.0}</horizontal_fov>
                     <image>
-                        <width>640</width>
-                        <height>480</height>
-                        <format>R8G8B8</format>
+                        <width>512</width>
+                        <height>424</height>
+                        <format>L8</format>
                     </image>
                     <clip>
-                        <near>0.01</near>
-                        <far>5.0</far>
+                        <near>0.1</near>
+                        <far>8.0</far>
                     </clip>
                     <noise>
@@ -93,4 +105,46 @@
             </sensor>
         </gazebo>
+        <gazebo reference="${name}_link">
+            <sensor name="${name}_camera" type="camera">
+                <always_on>true</always_on>
+                <update_rate>30.0</update_rate>
+                <camera name="${name}_camera">
+                    <horizontal_fov>${60*3.14/180.0}</horizontal_fov>
+                    <image>
+                        <width>1920</width>
+                        <height>1080</height>
+                        <format>R8G8B8</format>
+                    </image>
+                    <clip>
+                        <near>0.02</near>
+                        <far>10.0</far>
+                    </clip>
+                    <noise>
+                        <!-- Noise is sampled independently per pixel on each frame.
+                        That pixel's noise value is added to each of its color
+                        channels, which at that point lie in the range [0,1]. -->
+                        <type>gaussian</type>
+                        <mean>0.0</mean>
+                        <stddev>0.007</stddev>
+                    </noise>
+                </camera>
+                <plugin name="${name}_camera_controller"
+                        filename="libgazebo_ros_camera.so">
+                    <alwaysOn>true</alwaysOn>
+                    <update_rate>30.0</update_rate>
+                    <cameraName>${name}</cameraName>
+                    <imageTopicName>hd/image_color_rect</imageTopicName>
+                    <cameraInfoTopicName>hd/camera_info</cameraInfoTopicName>
+                    <frameName>${name}_rgb_optical_frame</frameName>
+                    <baseline>0.1</baseline>
+                    <distortionK1>0.0</distortionK1>
+                    <distortionK2>0.0</distortionK2>
+                    <distortionK3>0.0</distortionK3>
+                    <distortionT1>0.0</distortionT1>
+                    <distortionT2>0.0</distortionT2>
+                    <robotNamespace>${prefix}</robotNamespace>
+                </plugin>
+            </sensor>
+        </gazebo>
     </xacro:macro>
 </robot>

File: kinova_description/urdf/kinect_stand.urdf.xacro (robot description, xacro)
@@ -4,9 +4,9 @@
     <xacro:arg name="gazebo" default="false"/>
     <!-- Stand URDF -->
-    <xacro:include filename="$(find kinect_description)/urdf/stand/stand.urdf.xacro">
+    <xacro:include filename="$(find kinova_description)/urdf/stand/stand.urdf.xacro">
         <xacro:arg name="gazebo" value="${gazebo}"/>
     </xacro:include>
     <!-- Kinect URDF -->
-    <xacro:include filename="$(find kinect_description)/urdf/kinect/kinect.xacro">
+    <xacro:include filename="$(find kinova_description)/urdf/kinect/kinect.xacro">
         <xacro:arg name="gazebo" value="${gazebo}"/>
     </xacro:include>
@@ -14,9 +14,9 @@
                          name="kinect"
                          parent="sensor_link"
-                         cam_px="0.0"
-                         cam_py="0.05"
+                         cam_px="0.03"
+                         cam_py="0.015"
                          cam_pz="0.0"
                          cam_or="0.0"
-                         cam_op="${38*PI/180}"
+                         cam_op="${40*PI/180}"
                          cam_oy="0.0"/>
 </robot>

File: kinova_description/urdf/stand/properties.xacro (robot description, xacro)
@@ -6,5 +6,5 @@
     <xacro:property name="footMass" value="5.0"/>
     <xacro:property name="standRadius" value="0.03"/>
-    <xacro:property name="standHeight" value="1.5"/>
+    <xacro:property name="standHeight" value="1.3"/>
     <xacro:property name="standMass" value="0.5"/>
 </robot>

Commit message: Apriltags

File: kinova_description/urdf/kinect/kinect.xacro (robot description, xacro)
@@ -110,5 +110,5 @@
                 <update_rate>30.0</update_rate>
                 <camera name="${name}_camera">
-                    <horizontal_fov>${60*3.14/180.0}</horizontal_fov>
+                    <horizontal_fov>${70*3.14/180.0}</horizontal_fov>
                     <image>
                         <width>1920</width>

File: kinova_description/urdf/kinect_stand.urdf.xacro (robot description, xacro)
@@ -14,9 +14,9 @@
                          name="kinect"
                          parent="sensor_link"
-                         cam_px="0.03"
+                         cam_px="0.05"
                          cam_py="0.015"
                          cam_pz="0.0"
                          cam_or="0.0"
-                         cam_op="${45*PI/180}"
+                         cam_op="${60*PI/180}"
                          cam_oy="0.0"/>
 </robot>

File: kinova_description/urdf/stand/properties.xacro (robot description, xacro)
@@ -6,5 +6,5 @@
     <xacro:property name="footMass" value="5.0"/>
     <xacro:property name="standRadius" value="0.03"/>
-    <xacro:property name="standHeight" value="1.1"/>
+    <xacro:property name="standHeight" value="1.2"/>
     <xacro:property name="standMass" value="0.5"/>
 </robot>
